File: ha-pcb.kicad_sch (KiCad schematic)
At the start: 52 parts, among them J1 RJ45_NC1W, J10 1VAC_00, J11 1VAC_01, J12 5VCC_02, J13 5VCC_03, J14 30VCC_11, J15 ONOFF_134, J16 I2C_5V, J17 12VDC OUT, J2 RaPi_Connector, J3 RJ45_NC1W, J4 SainSmart_connector, J5 RJ45_1W1W, J6 RJ45_1W1W, J7 RJ45_1W1W, J8 RJ45_1W1W_T, J9 12VDC IN, U1 DMO063_SSR, U10 ADS1115 ADC, U11 ADS1115, U2 PCF_8575, U3 AK-DS2482S-100, U4 Pololu_Level_Shifter, U5 DS18B20, U6 PCA9615_I2C_Diff, U7 AK-DS2482S-100, U8 AK-DS2482S-100, U9 AK-DS2482S-100

Commit message: Incorporated feedback from forum.\nAdded two GPIOs for test marking
Parts:
- added JP1: Jumper_2_Open, Connector_PinHeader_2.54mm:PinHeader_1x02_P2.54mm_Vertical, symbol Jumper:Jumper_2_Open
- added R12, R13: 1K, Resistor_THT:R_Axial_DIN0207_L6.3mm_D2.5mm_P10.16mm_Horizontal, symbol Device:R
- C4: value 470uF -> 470uF/16V; footprint Capacitor_THT:CP_Radial_D6.3mm_P2.50mm -> Capacitor_THT:CP_Radial_D8.0mm_P3.80mm
- D1: value yellow -> LED; footprint LED_THT:LED_D5.0mm_IRGrey -> LED_THT:LED_D5.0mm
- D4, D5: value yellow -> LED
- J11: renamed from J8; value RJ45_1W1W_T -> RJ45_1W1W
- J12: renamed from J10; value 1VAC_00 -> 3.5Inch_Audio
- J13: renamed from J11; value 1VAC_01 -> 3.5Inch_Audio
- J14: renamed from J12; value 5VCC_02 -> 3.5Inch_Audio
- J15: renamed from J13; value 5VCC_03 -> 3.5Inch_Audio
- J16: renamed from J14; value 30VCC_11 -> 3.5Inch_Audio
- J17: renamed from J15; value ONOFF_134 -> 3.5Inch_Audio
- J2: renamed from J9; value 12VDC IN -> 12V IN
- J3: renamed from J17; value 12VDC OUT -> 12V OUT
- J6: renamed from J16; value I2C_5V -> Conn_01x05
- U6: renamed from U5; footprint Package_TO_SOT_THT:TO-92_Inline -> Package_TO_SOT_THT:TO-92_Inline_Wide
- U8: renamed from U10; value ADS1115 ADC -> ADS1115
- renumbered J7 to J10, J2 to J4, J3 to J5, J4 to J7, J5 to J8, J6 to J9, U8 to U10, U9 to U11, U4 to U2, U2 to U3, U3 to U4, U6 to U5, U11 to U9
Connections:
- net GND: now also J1.SH, J10.SH, J11.SH, J12.4 (GND), J12.5 (GND), J13.4 (GND), J13.5 (GND), J14.4 (GND), J14.5 (GND), J15.4 (GND), J15.5 (GND), J16.4 (GND), J16.5 (GND), J17.4 (GND), J17.5 (GND), J5.SH, J8.SH, J9.SH, R12.2, R13.2
- net A2/2: now reaches J17.2 (Tip), R6.1, U9.2 (Ain2)
- net A2/1: now reaches C3.1, C4.1, R7.1, R8.2, U9.3 (Ain1)
- net A1/2: now reaches D4.2 (A), R10.1, U8.2 (Ain2)
- net A1/3: now reaches D5.2 (A), R11.1, U8.1 (Ain3)
- net A1/1: now reaches J13.2 (Tip), U8.3 (Ain1)
- net A1/0: now reaches J12.2 (Tip), U8.4 (Ain0)
- net A2/3: now reaches J17.3 (Ring), R9.1, U9.1 (Ain3)
- net at J4.11 (GPIO17): now also R12.1
- net at J4.13 (GPIO27): now also JP1.2 (B)
- net 5VRB renamed A2/0
- new net: JP1.1 (A), R13.1
- no-connect marks 35 -> 33
Other:
- note added: "PWR from Raspberry (microUSB powered)"
- moved on the sheet: C1, C2, C3, C4, D2, D3, D4, D5, H1, H2, H3, H4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
